File: Hardware/Module - TPS540x/TPS540x2.kicad_sch (KiCad schematic)
At the start: 21 parts, among them J701 Jack-DC, J702 USB_A, J703 USB_C_Receptacle, J704 XT30, J705 USB_A+C, J706 XT30+Barrel, U701 TPS5403

Commit message: ...
Parts:
- added J707: USB-C_XT30, tinker:USB-C_XT30, symbol tinker:USB_A+C
- J706: now left out of the parts list
Connections:
- net GND: now also J707.4 (GND), J707.5 (Shield)
- net VoutB: now also J707.1 (VBUS)
- no-connect marks 12 -> 14
Changed lines of the file:
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@@
   (junction (at 143.51 27.94) (diameter 0) (color 0 0 0 0)
+  )
+  (junction (at 144.78 186.69) (diameter 0) (color 0 0 0 0)
   )
   (junction (at 66.04 30.48) (diameter 0) (color 0 0 0 0)
@@
   (no_connect (at 102.87 142.24))
   (no_connect (at 102.87 127))
+  (no_connect (at 135.89 175.26))
   (no_connect (at 102.87 134.62))
+  (no_connect (at 135.89 177.8))
   (no_connect (at 67.31 119.38))
   (no_connect (at 67.31 121.92))
@@
     (stroke (width 0) (type default) (color 0 0 0 0))
   )
+  (wire (pts (xy 146.05 185.42) (xy 146.05 186.69))
+    (stroke (width 0) (type default) (color 0 0 0 0))
+  )
   (wire (pts (xy 43.18 27.94) (xy 43.18 34.29))
     (stroke (width 0) (type default) (color 0 0 0 0))
@@
     (stroke (width 0) (type default) (color 0 0 0 0))
   )
+  (wire (pts (xy 143.51 186.69) (xy 144.78 186.69))
+    (stroke (width 0) (type default) (color 0 0 0 0))
+  )
   (wire (pts (xy 66.04 41.91) (xy 66.04 50.8))
     (stroke (width 0) (type default) (color 0 0 0 0))
@@
     (stroke (width 0) (type default) (color 0 0 0 0))
   )
+  (wire (pts (xy 143.51 185.42) (xy 143.51 186.69))
+    (stroke (width 0) (type default) (color 0 0 0 0))
+  )
   (wire (pts (xy 111.76 22.86) (xy 114.3 22.86))
     (stroke (width 0) (type default) (color 0 0 0 0))
@@
     (stroke (width 0) (type default) (color 0 0 0 0))
   )
+  (wire (pts (xy 146.05 186.69) (xy 144.78 186.69))
+    (stroke (width 0) (type default) (color 0 0 0 0))
+  )
   (wire (pts (xy 72.39 165.1) (xy 72.39 166.37))
     (stroke (width 0) (type default) (color 0 0 0 0))
@@
   (wire (pts (xy 66.04 30.48) (xy 66.04 34.29))
     (stroke (width 0) (type default) (color 0 0 0 0))
+  )
+  (text "Position:\n138,93.9" (at 156.21 182.88 0)
+    (effects (font (size 1.27 1.27) bold) (justify left bottom))
   )
   (text "Position:\n138,93.9" (at 86.36 162.56 0)
@@
     )
   )
+  (global_label "VoutB" (shape input) (at 135.89 170.18 180) (fields_autoplaced)
+    (effects (font (size 1.27 1.27)) (justify right))
+    (property "Intersheet References" "${INTERSHEET_REFS}" (id 0) (at 128.1834 170.1006 0)
+      (effects (font (size 1.27 1.27)) (justify right) hide)
+    )
+  )
   (global_label "VoutB" (shape input) (at 26.67 138.43 180) (fields_autoplaced)
     (effects (font (size 1.27 1.27)) (justify right))
@@
     (pin "2")
   )
+  (symbol (lib_id "power:GND") (at 144.78 186.69 0) (unit 1)
+    (in_bom yes) (on_board yes) (fields_autoplaced)
+    (property "Reference" "#PWR0105" (id 0) (at 144.78 193.04 0)
+      (effects (font (size 1.27 1.27)) hide)
+    )
+    (property "Value" "GND" (id 1) (at 144.78 191.77 0))
+    (property "Footprint" "" (id 2) (at 144.78 186.69 0)
+      (effects (font (size 1.27 1.27)) hide)
+    )
+    (property "Datasheet" "" (id 3) (at 144.78 186.69 0)
+      (effects (font (size 1.27 1.27)) hide)
+    )
+    (pin "1")
+  )
   (symbol (lib_id "Device:C") (at 119.38 24.13 0) (unit 1)
     (in_bom yes) (on_board yes) (fields_autoplaced)
@@
   )
   (symbol (lib_id "Connector_Generic_MountingPin:Conn_01x02_MountingPin") (at 31.75 158.75 0) (unit 1)
-    (in_bom yes) (on_board yes) (fields_autoplaced)
+    (in_bom no) (on_board no) (fields_autoplaced)
     (property "Reference" "J706" (id 0) (at 34.29 159.1055 0)
       (effects (font (size 1.27 1.27)) (justify left))
@@
     (pin "1")
   )
+  (symbol (lib_id "tinker:USB_A+C") (at 143.51 175.26 0) (mirror y) (unit 1)
+    (in_bom yes) (on_board yes)
+    (property "Reference" "J707" (id 0) (at 138.43 163.83 0)
+      (effects (font (size 1.27 1.27)) (justify right))
+    )
+    (property "Value" "USB-C_XT30" (id 1) (at 138.43 166.37 0)
+      (effects (font (size 1.27 1.27)) (justify right))
+    )
+    (property "Footprint" "tinker:USB-C_XT30" (id 2) (at 139.7 176.53 0)
+      (effects (font (size 1.27 1.27)) hide)
+    )
+    (property "Datasheet" " ~" (id 3) (at 139.7 176.53 0)
+      (effects (font (size 1.27 1.27)) hide)
+    )
+    (property "LCSC" "C6389922" (id 4) (at 143.51 175.26 0)
+      (effects (font (size 1.27 1.27)) hide)
+    )
+    (property "DigiKey" "AU-Y1005" (id 5) (at 143.51 175.26 0)
+      (effects (font (size 1.27 1.27)) hide)
+    )
+    (pin "1")
+    (pin "2")
+    (pin "3")
+    (pin "4")
+    (pin "5")
+    (pin "A5")
+    (pin "A8")
+    (pin "B5")
+    (pin "B8")
+  )
   (symbol (lib_id "power:GND") (at 119.38 35.56 0) (unit 1)
