File: Hardware/Module - TPS540x/Module - TPS540x.kicad_pcb (KiCad board)
At the start: 2 copper layers, 100 x 40 mm, 89 parts, among them J505 USB_A+C, J706 XT30+Barrel, Q401 ZXMP4A16G, Q601 ZXMP4A16G, U1 ATtiny1617, U501 TPS5403, U701 TPS5403

Commit message: ...
Parts:
- removed J706: XT30+Barrel, tinker:CONN-TH_XT30PW-F-1+Barrel
- added J707: USB-C_XT30, tinker:USB-C_XT30, F.Cu at (138.0, 90.0)

Commit message: .
Parts:
- removed C401: 330uF, Capacitor_SMD:CP_Elec_10x10
- removed C402: 10uF, Capacitor_SMD:C_1206_3216Metric
- removed C403, C701: 100nF, Capacitor_SMD:C_0603_1608Metric
- removed C703: 100pF, Capacitor_SMD:C_0603_1608Metric
- removed C704: 10nF, Capacitor_SMD:C_0603_1608Metric
- removed C705: 330uF, Capacitor_SMD:CP_Elec_8x10
- removed C706: 2.2nF, Capacitor_SMD:C_0603_1608Metric
- removed D701: LED, LED_SMD:LED_0603_1608Metric
- removed D702: DSK24, Diode_SMD:D_SOD-123
- removed F701: Polyfuse, tinker:F1206
- removed J505: USB_A+C, tinker:USB_A+C
- removed J707: USB-C_XT30, tinker:USB-C_XT30
- removed L701: L_Ferrite, tinker:IND-SMD_L7.1-W6.6
- removed Q601: ZXMP4A16G, tinker:SOT-223-3_TabPin2_opt23
- removed R701: ?, Resistor_SMD:R_0603_1608Metric
- removed R702: 100K, Resistor_SMD:R_0603_1608Metric
- removed R703: 47K, Resistor_SMD:R_0603_1608Metric
- removed the TP1 at (79.5, 114.0)
- removed the TP4 at (77.0, 114.0)
- removed TP502: Vout1, tinker:TestPoint_THTPad_D1.0mm_Drill0.5mm
- removed TP701: VswB, tinker:TestPoint_THTPad_D1.0mm_Drill0.5mm
- removed TP702: VoutB, tinker:TestPoint_THTPad_D1.0mm_Drill0.5mm
- removed TPa0: ~{RESET}, tinker:TestPoint_THTPad_D1.0mm_Drill0.5mm
- removed TPa401, TPa602: CtrlA, tinker:TestPoint_THTPad_D1.0mm_Drill0.5mm
- removed U701: TPS5403, Package_SO:SOIC-8_3.9x4.9mm_P1.27mm
- added C1: 220uF, Capacitor_SMD:CP_Elec_10x10, F.Cu at (73.0, 91.0)
- added C2: 10uF, Capacitor_SMD:C_1206_3216Metric, F.Cu at (66.0, 94.0)
- added C3: 100nF, Capacitor_SMD:C_0603_1608Metric, F.Cu at (73.0, 83.5)
- added C502: 100nF, Capacitor_SMD:C_0603_1608Metric, F.Cu at (98.1, 84.6)
- added C507: 330uF, Capacitor_SMD:CP_Elec_8x10, F.Cu at (123.8, 93.0)
- added C604: 100pF, Capacitor_SMD:C_0603_1608Metric, F.Cu at (99.0, 109.3)
- added C605: 10nF, Capacitor_SMD:C_0603_1608Metric, F.Cu at (99.0, 107.8)
- added C606: 2.2nF, Capacitor_SMD:C_0603_1608Metric, F.Cu at (99.0, 112.3)
- added C607: 330uF, Capacitor_SMD:CP_Elec_8x10, F.Cu at (123.8, 112.0)
- added D601: LED, LED_SMD:LED_0603_1608Metric, F.Cu at (147.9, 100.9)
- added D602: DSK24, Diode_SMD:D_SOD-123, F.Cu at (111.3, 104.6)
- added F602: Polyfuse, tinker:F1206, F.Cu at (131.2, 112.0)
- added J201: UPDI Connection, tinker:UPDI_connection, F.Cu at (71.0, 114.0)
- added J507: USB_A+C+XT30, tinker:USB_A+C+XT30, F.Cu at (150.0, 90.5)
- added J607: USB_A+C+XT30, tinker:USB_A+C+XT30, F.Cu at (150.0, 109.5)
- added JP201: Jumper_2_Bridged, tinker:tinySJ-Bridged, F.Cu at (75.0, 110.3)
- added L601: L_Ferrite, tinker:IND-SMD_L7.1-W6.6, F.Cu at (115.9, 105.8)
- added PA0: CtrlA, tinker:TestPoint_THTPad_D1.0mm_Drill0.5mm, F.Cu at (89.0, 114.0)
- added Q301: ZXMP4A16G, Package_TO_SOT_SMD:SOT-223-3_TabPin2, F.Cu at (86.7, 86.0)
- added R301: 100R, Resistor_SMD:R_0603_1608Metric, F.Cu at (80.7, 86.0)
- added R302: 10k, Resistor_SMD:R_0603_1608Metric, F.Cu at (80.7, 83.7)
- added R603: 47K, Resistor_SMD:R_0603_1608Metric, F.Cu at (99.0, 110.8)
- added TP301: CtrlA, tinker:TestPoint_THTPad_D1.0mm_Drill0.5mm, F.Cu at (79.9, 88.3)
- added TP302: VswA, tinker:TestPoint_THTPad_D1.0mm_Drill0.5mm, F.Cu at (92.2, 86.0)
- added TP401: CtrlA, tinker:TestPoint_THTPad_D1.0mm_Drill0.5mm, F.Cu at (79.9, 95.6)
- added TP402: VswB, tinker:TestPoint_THTPad_D1.0mm_Drill0.5mm, F.Cu at (92.2, 93.3)
- added TP601: Vout1, tinker:TestPoint_THTPad_D1.0mm_Drill0.5mm, F.Cu at (133.5, 115.0)
- added U601: TPS5403, Package_SO:SOIC-8_3.9x4.9mm_P1.27mm, F.Cu at (105.3, 105.6)
- C501: value 100nF -> 10uF; footprint Capacitor_SMD:C_0603_1608Metric -> Capacitor_SMD:C_1206_3216Metric
- C503: value 100pF -> 100nF
- C504: value 10nF -> 100pF
- C505: value 330uF -> 10nF; footprint Capacitor_SMD:CP_Elec_8x10 -> Capacitor_SMD:C_0603_1608Metric
- C601: value 330uF -> 10uF; footprint Capacitor_SMD:CP_Elec_10x10 -> Capacitor_SMD:C_1206_3216Metric
- C602: value 10uF -> 100nF; footprint Capacitor_SMD:C_1206_3216Metric -> Capacitor_SMD:C_0603_1608Metric
- Q401: footprint tinker:SOT-223-3_TabPin2_opt23 -> Package_TO_SOT_SMD:SOT-223-3_TabPin2
- R601: value 100R -> ?
- R602: value 10k -> 100K
- TP501: value VswA -> Vout1
- moved R601 77.8 mm to (144.9, 100.9), turned to 0 degrees
- moved R602 36.1 mm to (99.0, 106.2), turned to 180 degrees
- moved C503 33.5 mm to (105.3, 83.0), turned to 0 degrees
- moved TP501 31.9 mm to (133.5, 96.0)
- moved C505 31.5 mm to (99.0, 88.8), turned to 180 degrees
- moved R502 30.1 mm to (99.0, 87.3), turned to 180 degrees
- moved C504 26.7 mm to (99.0, 90.3), turned to 180 degrees
- moved C506 26.7 mm to (99.0, 93.4), turned to 0 degrees
- moved PB0 26.0 mm to (73.0, 100.0), turned to 90 degrees
- moved C501 25.8 mm to (95.5, 84.5), turned to 90 degrees
- moved R503 25.6 mm to (99.0, 91.8), turned to 180 degrees
- moved PB1 24.1 mm to (75.0, 100.0), turned to 90 degrees
- moved U501 23.5 mm to (105.3, 86.6)
- moved PB2 22.4 mm to (77.0, 100.0), turned to 90 degrees
- moved PB3 20.9 mm to (79.0, 100.0), turned to 90 degrees
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- renumbered C1 to C4, C2 to C5, D301 to D1, F301 to F1, TPa1 to PA1, TPa2 to PA2, TPa3 to PA3, TPa4 to PA4, TPa5 to PA5, TPa6 to PA6, TPa7 to PA7, TPb0 to PB0, TPb1 to PB1, TPb2 to PB2, TPb3 to PB3, TPb4 to PB4, TPb5 to PB5, TPb6 to PB6, TPb7 to PB7, TPc0 to PC0, TPc1 to PC1, TPc2 to PC2, TPc3 to PC3, TPc4 to PC4, TPc5 to PC5, R3 to R1, R4 to R2, R1 to R3, R2 to R4, TP301 to TP1, TP302 to TP2, TP5 to TP3, TP6 to TP4, TP7 to TP5, TP8 to TP6, TP303 to TP7
Connections:
- net /ATTinyXX17/PA0 renamed PA0
- net /TPS540x 1/ROSC A renamed /TPS540x-A/ROSC A
- C501 pad 1: /TPS540x 1/BOOT A -> VswA
- C501 pad 2: /TPS540x 1/LX -> GND
- C503 pad 1: /TPS540x 1/COMP A -> /TPS540x-A/BOOT A
- C503 pad 2: GND -> /TPS540x-A/LX
- C504 pad 1: Net-(C504-Pad1) -> /TPS540x-A/COMP A
- C505 pad 1: /TPS540x 1/Vsense A -> Net-(C505-Pad1)
- C603 pad 1: VswB -> /TPS540x-B/BOOT A
- C603 pad 2: GND -> /TPS540x-B/LX
- D502 pad 1: /TPS540x 1/LX -> /TPS540x-A/LX
- F501 pad 1: /TPS540x 1/Vsense A -> /TPS540x-A/Vsense A
- L501 pad 1: /TPS540x 1/LX -> /TPS540x-A/LX
- L501 pad 2: /TPS540x 1/Vsense A -> /TPS540x-A/Vsense A
- Q401 pad 2: VswA -> VswB
- R401 pad 1: PA1 -> PB5
- R503 pad 1: /TPS540x 1/COMP A -> /TPS540x-A/COMP A
- R601 pad 1: PA2 -> VoutB
- R601 pad 2: Net-(Q601-Pad1) -> Net-(D601-Pad2)
- R602 pad 1: Vin -> /TPS540x-B/ROSC A
- R602 pad 2: Net-(Q601-Pad1) -> GND
- TP501 pad 1: VswA -> VoutA
- U501 pad 1: /TPS540x 1/BOOT A -> /TPS540x-A/BOOT A
- U501 pad 4: Net-(C504-Pad1) -> Net-(C505-Pad1)
- U501 pad 5: /TPS540x 1/Vsense A -> /TPS540x-A/Vsense A
- U501 pad 6: /TPS540x 1/COMP A -> /TPS540x-A/COMP A
- U501 pad 8: /TPS540x 1/LX -> /TPS540x-A/LX
Routing:
- net PA2: track 43.4 -> 5.79 mm, vias 1 -> 0
- net VswA: track 55.2 -> 19.2 mm, vias 2 -> 0
- net PA1: track 40.2 -> 7.02 mm, vias 1 -> 0
- net I2C-Vcc: track 1.65 -> 30.5 mm, vias 1 -> 2
- net PB1: track 54.3 -> 32.8 mm, vias 4 -> 3
- net GND: track 6.95 -> 23.2 mm, vias 29 -> 19
- net PA0: track 6.93 -> 22.1 mm, vias 0 -> 2
- net VswB: track 43.4 -> 29.8 mm, vias 2 -> 0
- net /TPS540x 1/LX: track 11.7 -> 0.00 mm
- net /TPS540x-A/LX: track 0.00 -> 10.9 mm
- net /TPS540x-B/LX: track 0.00 -> 10.9 mm
- net /TPS540x 2/LX: track 10.9 -> 0.00 mm
- net /TPS540x-B/COMP A: track 0.00 -> 10.8 mm
- net /TPS540x-A/COMP A: track 0.00 -> 10.8 mm
- net PC2: track 15.8 -> 5.17 mm, vias 1 -> 0
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- added copper zone on F.Cu, net /TPS540x-A/Vsense A
- added copper zone on F.Cu, net /TPS540x-B/Vsense A
- removed copper zone on F.Cu, net /TPS540x 1/Vsense A
- removed copper zone on F.Cu, net /TPS540x 2/Vsense B
- removed copper zone on F.Cu, net VswA
- removed copper zone on F.Cu, net VswB
Other:
- board text added: "${COMMENT1}"
- board text added: "${COMMENT2} (v${REVISION})"
- board text added: "0"
- board text added: "A"
- board text added: "ATTiny XXx7"
- board text added: "B"
- board text added: "Bridge to Bypass"
- board text added: "Cut to Isolate"
- board text added: "Incoming Power Section"
- board text added: "Output Section A"
- board text added: "Output Section B"
- board text added: "Overkill Central! :P"
- board text added: "PA0"
- board text added: "PortA"
- board text added: "PortB"
- board text added: "PortC"
- board text added: "Power Control Section"
- board text added: "RxD"
- board text added: "TxD"
- board text added: "Vcc (3v3)"
- board text added: "Voltage A:"
- board text added: "Voltage B:"
- board text added: "~{RST} (global)"
- board text removed: "${COMMENT1} - ${COMMENT2} (v${REVISION})"
- board text removed: "(RxD)"
- board text removed: "(SCL)"
- board text removed: "(SDA)"
- board text removed: "(TxD)"
- board text removed: "100"
- board text removed: "106.426"
- board text removed: "106.934"
- board text removed: "109.6"
- board text removed: "110"
- board text removed: "113.1"
- board text removed: "115.57"
- board text removed: "116.078"
- board text removed: "138"
- board text removed: "87.226"
- board text removed: "87.734"
- board text removed: "90"
- board text removed: "90.4"
- board text removed: "93.9"
- board text removed: "96.37"
- board text removed: "96.878"
- board text removed: "ATTiny XX17"
- board text removed: "Dat0"
- board text removed: "PA1"
- board text removed: "PA2"
- board text removed: "UPDI"
- board text removed: "Unified Program R & + - Debug Interface"
