File: Hardware/Module - TPS540x/Module - TPS540x.kicad_sch (KiCad schematic)
At the start: 0 parts

Commit message: .
Other:
- removed sheet TPS540x 1
- removed sheet TPS540x 2
- added sheet TPS540x-A (TPS540x-A.kicad_sch)
- added sheet TPS540x-B (TPS540x-B.kicad_sch)
