File: Hardware/Tool - ATTiny Module Flasher/Tool - ATTiny Module Flasher.kicad_pcb (KiCad board)
At the start: 2 copper layers, 50 x 20 mm, 20 parts, among them J102 USB_C_Receptacle, J902 Conn_01x03, SW202 SW_DIP_x01, U202 AMS1117-3.3, U303 CH340C

Commit message: .
Parts:
- moved G*** 28.7 mm to (106.5, 93.0), turned to 90 degrees
- moved REF** 14.5 mm to (106.5, 107.0), turned to 90 degrees
Other:
- board size 50 x 20 mm -> 60 x 20 mm
