File: Hardware/Tool - ATTiny Module Flasher/Tool - ATTiny Module Flasher.kicad_pcb (KiCad board)
At the start: 2 copper layers, 60 x 20 mm, 20 parts, among them J102 USB_C_Receptacle, J902 Conn_01x03, SW202 SW_DIP_x01, U202 AMS1117-3.3, U303 CH340C

Commit message: updating tools designs
Parts:
- J902: footprint tinker:PinHeader_1x03_P2.54mm_Horizontal -> tinker:UPDI-Pogo
- moved J902 5.08 mm to (104.0, 97.5), turned to 0 degrees
Other:
- board size 60 x 20 mm -> 61.5 x 20 mm
- board text removed: "GND"
- board text removed: "UPDI"
- board text removed: "Vcc"
- board text removed: "~{RST}"
