File: Hardware/Tool - ATTiny Module Flasher/UPDI.kicad_sch (KiCad schematic)
At the start: 5 parts, among them J902 Conn_01x03

Commit message: updating tools designs
Parts:
- J902: footprint tinker:PinHeader_1x03_P2.54mm_Horizontal -> tinker:UPDI-Pogo
Changed lines of the file:
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@@
     (property "Reference" "J902" (id 0) (at 78.74 57.15 0))
     (property "Value" "Conn_01x03" (id 1) (at 78.74 59.69 0))
-    (property "Footprint" "tinker:PinHeader_1x03_P2.54mm_Horizontal" (id 2) (at 78.74 66.04 0)
+    (property "Footprint" "tinker:UPDI-Pogo" (id 2) (at 78.74 66.04 0)
       (effects (font (size 1.27 1.27)) hide)
     )
