File: Hardware/Tool - ESP Module Flasher/Tool - ESP Module Flasher.kicad_pcb (KiCad board)
At the start: 2 copper layers, 50 x 20 mm, 21 parts, among them J102 USB_C_Receptacle, J802 Conn_01x06, Q801 MMBT3904, Q802 MMBT3904, SW202 SW_DIP_x01, U202 AMS1117-3.3, U303 CH340C

Commit message: .
Other:
- board size 50 x 20 mm -> 60 x 20 mm
