File: Hardware/Controller - ATTiny/Controller - ATTiny.kicad_pcb (KiCad board)
At the start: 2 copper layers, 100 x 40 mm, 58 parts, among them J1 USB_C_Receptacle, SW504 SW_DIP_x01, U1 ATtiny1617, U501 CH340C, U502 CD4053B

Commit message: Added a reset button to ATTiny controller board
Parts:
- added SW1: SW_Push, tinker:SW_Push_TS273014TP, F.Cu at (108.4, 115.1)
Routing:
- net ~{RESET}: track 46.6 -> 51.0 mm, vias 1 -> 2
Other:
- board text added: "RESET"
